File: schematic/Andy_Robot_Board/Andy.kicad_pcb (KiCad board)
At the start: 2 copper layers, 104.1 x 80 mm, 45 parts, among them K1 Servo, K10 Servo, K2 Servo, K3 Servo, K4 Servo, K5 Servo, K6 Servo, K7 Servo, K8 Servo, K9 Servo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

Commit message: Worked on PCB
Parts:
- added G***: LOGO, RobotLogo, F.Cu at (168.7, 196.3)
- added G***: LOGO, OpenSource, B.Cu at (161.5, 197.6)
- K1: value Servo -> Servo Header
- P1: value R-Pi Header -> Raspberry Pi
- P2: value Power Jumper -> Power
- P4: value GND Pins -> GND
Routing:
- net N-000002: track 0.00 -> 59.4 mm, vias 0 -> 2
- net N-0000051: track 0.00 -> 52.6 mm
- net GND: track 182.5 -> 231.9 mm, vias 0 -> 8
- net N-0000010: track 0.00 -> 45.4 mm, vias 0 -> 2
- net (no net): track 37.4 -> 0.00 mm, vias 1 -> 0
- net N-0000019: track 0.00 -> 35.6 mm, vias 0 -> 2
- net N-000008: track 59.0 -> 27.1 mm
- net N-0000017: track 0.00 -> 25.6 mm, vias 0 -> 2
- net N-0000018: track 0.00 -> 24.7 mm, vias 0 -> 2
- net N-0000072: track 43.3 -> 21.4 mm, vias 2 -> 1
- net N-0000033: track 35.8 -> 54.2 mm, vias 0 -> 1
- net N-0000016: track 0.00 -> 17.9 mm, vias 0 -> 4
- net N-0000079: track 113.9 -> 96.7 mm
- net N-0000071: track 38.1 -> 23.3 mm
- net N-0000027: track 31.1 -> 45.3 mm, vias 0 -> 2
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Other:
- board size 104.1 x 80 mm -> 104.1 x 56.9 mm
- board text added: "ANDY Robot Board"
- board text added: "Tyler Spadgenske"
- board text added: "Version 1.0"
